File: hw/pavapro3c.brd (EAGLE design)
At the start: 105 x 66 mm, 86 parts, among them IC1 ATmega328P, IC2 MIC5225-3.3v, IC3 PCF8574SOW, IC4 MAX3232-SOIC, Q1 reset, Y1 12MHz

Commit message: ver 3
Parts:
- removed D1, D4, D5, D6: 1N4148SOD, _mcom5:SOD-80
- added R28, R29: 3k3, microbuilder:_0805
- D7, D8: value 1N4148SOD -> BAT48
- R1, R2: value 68 (0603) -> 68
- R10, R11, R12, R13, R14: value 470 (0603) -> 1k
- R15, R16, R17, R18, R19: value 470 (0603) -> 100k
- R20, R21, R22, R23, R24: value 470 (0603) -> 150
- R25, R26, R27, R7: value 470 (0603) -> 10k
- R3: value 1.5K (0603) -> 1.5K
- R4, R5: value 470 (0603) -> 470
- R6: value 10K (0603) -> 10K
- R8, R9: value 470 (0603) -> DNP
Connections:
- net N$29 renamed MISO
- net N$30 renamed SCK
- net N$31 renamed RST
- removed net N$12: D1.A, IC3.12
- removed net N$13: D4.A, IC3.11
- removed net N$14: D5.A, IC3.10
- removed net N$15: D6.A, IC3.9
- removed net N$25: R10.2, SV1.4
- removed net N$27: R11.2, SV1.2
- new net MOSI: R11.2, SV1.4
- new net VCC: R10.2, SV1.2
- net +3V3: now also R28.2, R29.2, U$5.8; no longer U$5.7
- net A4: now also R28.1
- net A5: now also R29.1
- net GND: now also U$5.7; no longer U$5.8
- net N$10: now also IC3.10; no longer D5.K
- net N$11: now also IC3.9; no longer D6.K
- net N$8: now also IC3.12; no longer D1.K
- net N$9: now also IC3.11; no longer D4.K
Routing:
- net N$27: track 18.2 -> 0.00 mm
- net MOSI: track 0.00 -> 12.7 mm
- net N$8: track 5.67 -> 18.2 mm
- net VCC: track 0.00 -> 12.0 mm
- net N$9: track 5.48 -> 17.4 mm
- net N$10: track 5.16 -> 16.8 mm
- net N$12: track 11.2 -> 0.00 mm
- net N$25: track 9.91 -> 0.00 mm
- net +3V3: track 221.7 -> 231.4 mm
- net N$13: track 9.36 -> 0.00 mm
- net N$11: track 5.03 -> 14.4 mm
- net N$14: track 8.96 -> 0.00 mm
- net A5: track 117.0 -> 125.8 mm
- net N$15: track 6.05 -> 0.00 mm
- net A4: track 127.1 -> 131.8 mm
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